Commit message: Adds packages installation

File: sr_description/urdf/macros.xacro (robot description, xacro)
@@ -37,5 +37,5 @@
     </joint>
     <actuator name="${name}_act">
-      <hardwareInterface>hardware_interface/VelocityJointInterface</hardwareInterface>
+      <!-- <hardwareInterface>hardware_interface/VelocityJointInterface</hardwareInterface> -->
       <mechanicalReduction>1</mechanicalReduction>
     </actuator>
@@ -84,5 +84,5 @@
       <material name="white"/>
     </visual>
-    <xacro:box_inertial mass="${mass/10.0}" x="${offset}" y="${radius}" z="${radius}">
+    <xacro:box_inertial mass="${mass*0.5}" x="${offset}" y="${radius}" z="${radius}">
       <origin xyz="${-offset/2.0} 0 0" rpy="0 0 0" />
     </xacro:box_inertial>
@@ -109,5 +109,5 @@
       <material name="wheel"/>
     </visual>
-    <xacro:sphere_inertial mass="${9.0/10.0*mass}" radius="${radius}">
+    <xacro:sphere_inertial mass="${mass*0.5}" radius="${radius}">
       <origin xyz="0 0 0" rpy="0 0 0" />
     </xacro:sphere_inertial>

File: sr_description/urdf/sr_robot.xacro (robot description, xacro)
@@ -9,9 +9,9 @@
   <xacro:property name="PI" value="3.1415926535897931"/>
   <!-- Wheels constants -->
-  <xacro:property name="wheel_mass" value="3"/>
+  <xacro:property name="wheel_mass" value="8"/>
   <xacro:property name="wheel_radius" value="0.25"/>
   <xacro:property name="wheel_width" value="0.1"/>
   <!-- Chassis constants -->
-  <xacro:property name="chassis_mass" value="60"/>
+  <xacro:property name="chassis_mass" value="12"/>
   <xacro:property name="chassis_lenght" value="0.95"/>
   <xacro:property name="chassis_width" value="0.5"/>
@@ -22,5 +22,5 @@
   <xacro:property name="axle_offset" value="${chassis_lenght/2-wheel_radius}"/>
   <!-- Caster wheel -->
-  <xacro:property name="caster_mass" value="1"/>
+  <xacro:property name="caster_mass" value="8"/>
   <xacro:property name="caster_radius" value="${clearence/2.0}"/>
   <xacro:property name="caster_offset" value="${caster_radius*1.5}"/>

Commit message: Dodaje kamerę do modelu

File: sr_description/urdf/macros.xacro (robot description, xacro)
@@ -46,5 +46,5 @@
   <link name="${name}_link">
     <collision>
-      <origin xyz="${-axle_offset} 0 ${height/2.0 + clearence}" rpy="0 0 0"/>
+      <origin xyz="${-axle_offset} 0 0" rpy="0 0 0"/>
       <geometry>
         <box size="${lenght} ${width} ${height}"/>
@@ -52,5 +52,5 @@
     </collision>
     <visual>
-      <origin xyz="${-axle_offset} 0 ${height/2.0 + clearence}" rpy="0 0 0"/>
+      <origin xyz="${-axle_offset} 0 0" rpy="0 0 0"/>
       <geometry>
         <box size="${lenght} ${width} ${height}"/>
@@ -59,5 +59,5 @@
     </visual>
     <xacro:box_inertial mass="${mass}" x="${lenght}" y="${width}" z="${height}">
-      <origin xyz="${-axle_offset} 0 ${height/2.0 + clearence}" rpy="0 0 0" />
+      <origin xyz="${-axle_offset} 0 0" rpy="0 0 0" />
     </xacro:box_inertial>
   </link>
@@ -65,5 +65,5 @@
     <parent link="${robot_name}/base_footprint"/>
     <child link="${name}_link"/>
-    <origin xyz="0 0 0" rpy="0 0 0"/>
+    <origin xyz="0 0 ${height/2.0 + clearence}" rpy="0 0 0"/>
   </joint>
 </xacro:macro>

File: sr_description/urdf/sr_robot.xacro (robot description, xacro)
@@ -21,4 +21,5 @@
   <xacro:property name="separation" value="${chassis_width+wheel_width+0.05}"/>
   <xacro:property name="axle_offset" value="${chassis_lenght/2-wheel_radius}"/>
+  <!-- <xacro:property name="axle_offset" value="0"/> -->
   <!-- Caster wheel -->
   <xacro:property name="caster_mass" value="8"/>
@@ -62,3 +63,10 @@
     <origin xyz="0.0 0.0 0.0" rpy="0 0 0" />
   </joint>
+  <!-- Camera -->
+  <link name="${robot_name}/camera_link" />
+  <joint name="${robot_name}/camera_joint" type="fixed">
+    <parent link="${robot_name}/base_link" />
+    <child link="${robot_name}/camera_link" />
+    <origin xyz="${chassis_lenght/2.0-axle_offset+0.05} 0.0 0.0" rpy="0 0 0" />
+  </joint>
 </robot>

Commit message: worlds and navigation

File: sr_description/urdf/macros.xacro (robot description, xacro)
@@ -1,123 +1,123 @@
 <?xml version="1.0"?>
 <robot xmlns:xacro="http://www.ros.org/wiki/xacro">
-<xacro:include filename="$(find sr_description)/urdf/inertials.xacro" />
-<xacro:include filename="$(find sr_description)/urdf/materials.xacro" />
-<!-- Wheel Joint and Link definition MACRO -->
-<xacro:macro name="wheel" params="name radius width mass dx dy">
-  <link name="${name}_link">
-    <collision>
-      <origin xyz="0 0 0" rpy="0 0 0"/>
-      <geometry>
-        <cylinder radius="${radius}" length="${width}"/>
-      </geometry>
-    </collision>
-    <visual>
-      <origin xyz="0 0 0" rpy="0 0 0"/>
-      <geometry>
+  <xacro:include filename="$(find sr_description)/urdf/inertials.xacro" />
+  <xacro:include filename="$(find sr_description)/urdf/materials.xacro" />
+  <!-- Wheel Joint and Link definition MACRO -->
+  <xacro:macro name="wheel" params="name radius width mass dx dy">
+    <link name="${name}_link">
+      <collision>
+        <origin xyz="0 0 0" rpy="0 0 0"/>
+        <geometry>
           <cylinder radius="${radius}" length="${width}"/>
-      </geometry>
-      <material name="wheel"/>
-    </visual>
-    <xacro:cylinder_inertial mass="${mass}" radius="${radius}" length="${width}">
-      <origin xyz="0 0 0" rpy="0 0 0"/>
-    </xacro:cylinder_inertial>
-  </link>
-  <joint name="${name}_joint" type="continuous">
-    <parent link="${robot_name}/base_footprint"/>
-    <child link="${name}_link"/>
-    <origin xyz="${dx} ${dy} ${wheel_radius}" rpy="${-PI/2.0} 0 0"/>
-    <axis xyz="0 0 1"/>
-    <limit effort="10000" velocity="20.0" />
-    <dynamics damping="0" friction="00"/>
-  </joint>
-  <transmission name="${name}_trans">
-    <type>transmission_interface/SimpleTransmission</type>
-    <joint name="${name}_joint">
-      <hardwareInterface>hardware_interface/VelocityJointInterface</hardwareInterface>
+        </geometry>
+      </collision>
+      <visual>
+        <origin xyz="0 0 0" rpy="0 0 0"/>
+        <geometry>
+          <cylinder radius="${radius}" length="${width}"/>
+        </geometry>
+        <material name="wheel"/>
+      </visual>
+      <xacro:cylinder_inertial mass="${mass}" radius="${radius}" length="${width}">
+        <origin xyz="0 0 0" rpy="0 0 0"/>
+      </xacro:cylinder_inertial>
+    </link>
+    <joint name="${name}_joint" type="continuous">
+      <parent link="${robot_name}/base_footprint"/>
+      <child link="${name}_link"/>
+      <origin xyz="${dx} ${dy} ${wheel_radius}" rpy="${-PI/2.0} 0 0"/>
+      <axis xyz="0 0 1"/>
+      <limit effort="-1" velocity="-1" />
+      <dynamics damping="0.0" friction="10"/>
     </joint>
-    <actuator name="${name}_act">
-      <!-- <hardwareInterface>hardware_interface/VelocityJointInterface</hardwareInterface> -->
-      <mechanicalReduction>1</mechanicalReduction>
-    </actuator>
-  </transmission>
-</xacro:macro>
-<!-- Chassis Joint and Link definition MACRO -->
-<xacro:macro name="chassis" params="name lenght width height axle_offset clearence mass">
-  <link name="${name}_link">
-    <collision>
-      <origin xyz="${-axle_offset} 0 0" rpy="0 0 0"/>
-      <geometry>
-        <box size="${lenght} ${width} ${height}"/>
-      </geometry>
-    </collision>
-    <visual>
-      <origin xyz="${-axle_offset} 0 0" rpy="0 0 0"/>
-      <geometry>
-        <box size="${lenght} ${width} ${height}"/>
-      </geometry>
-      <material name="chassis"/>
-    </visual>
-    <xacro:box_inertial mass="${mass}" x="${lenght}" y="${width}" z="${height}">
-      <origin xyz="${-axle_offset} 0 0" rpy="0 0 0" />
-    </xacro:box_inertial>
-  </link>
-  <joint name="${name}_joint" type="fixed">
-    <parent link="${robot_name}/base_footprint"/>
-    <child link="${name}_link"/>
-    <origin xyz="0 0 ${height/2.0 + clearence}" rpy="0 0 0"/>
-  </joint>
-</xacro:macro>
-<!-- Caster wheel joint and Link definition MACRO -->
-<xacro:macro name="caster" params="name radius mass offset dx">
-  <link name="${name}_rotation_link">
-    <collision>
-      <origin xyz="${-offset/2.0} 0 0" rpy="0 0 0" />
-      <geometry>
-        <box size="${offset} ${radius} ${radius}"/>
-      </geometry>
-    </collision>
-    <visual>
-      <origin xyz="${-offset/2.0} 0 0" rpy="0 0 0" />
-      <geometry>
-        <box size="${offset} ${radius} ${radius}"/>
-      </geometry>
-      <material name="white"/>
-    </visual>
-    <xacro:box_inertial mass="${mass*0.5}" x="${offset}" y="${radius}" z="${radius}">
-      <origin xyz="${-offset/2.0} 0 0" rpy="0 0 0" />
-    </xacro:box_inertial>
-  </link>
-  <joint name="${name}_rotation_joint" type="continuous">
-    <parent link="${robot_name}/base_footprint"/>
-    <child link="${name}_rotation_link"/>
-    <origin xyz="${dx} 0 ${1.5*caster_radius}" rpy="0 0 0"/>
-    <axis xyz="0 0 1"/>
-    <dynamics damping="0.01" friction="0.1"/>
-  </joint>
-  <link name="${name}_wheel_link">
-    <collision>
-      <origin xyz="0 0 0" rpy="0 0 0"/>
-      <geometry>
-        <sphere radius="${radius}"/>
-      </geometry>
-    </collision>
-    <visual>
-      <origin xyz="0 0 0" rpy="0 0 0"/>
-      <geometry>
-        <sphere radius="${radius}"/>
-      </geometry>
-      <material name="wheel"/>
-    </visual>
-    <xacro:sphere_inertial mass="${mass*0.5}" radius="${radius}">
-      <origin xyz="0 0 0" rpy="0 0 0" />
-    </xacro:sphere_inertial>
-  </link>
-  <joint name="${name}_wheel_joint" type="continuous">
-    <parent link="${name}_rotation_link"/>
-    <child link="${name}_wheel_link"/>
-    <origin xyz="${-offset} 0 ${-caster_radius / 2.0}" rpy="${-PI/2.0} 0 0"/>
-    <axis xyz="0 0 1"/>
-    <dynamics damping="0.01" friction="1.5"/>
-  </joint>
-</xacro:macro>
+    <transmission name="${name}_trans">
+      <type>transmission_interface/SimpleTransmission</type>
+      <joint name="${name}_joint">
+        <hardwareInterface>hardware_interface/VelocityJointInterface</hardwareInterface>
+      </joint>
+      <actuator name="${name}_act">
+        <hardwareInterface>hardware_interface/VelocityJointInterface</hardwareInterface>
+        <mechanicalReduction>1</mechanicalReduction>
+      </actuator>
+    </transmission>
+  </xacro:macro>
+  <!-- Chassis Joint and Link definition MACRO -->
+  <xacro:macro name="chassis" params="name lenght width height axle_offset clearence mass">
+    <link name="${name}_link">
+      <collision>
+        <origin xyz="${-axle_offset} 0 0" rpy="0 0 0"/>
+        <geometry>
+          <box size="${lenght} ${width} ${height}"/>
+        </geometry>
+      </collision>
+      <visual>
+        <origin xyz="${-axle_offset} 0 0" rpy="0 0 0"/>
+        <geometry>
+          <box size="${lenght} ${width} ${height}"/>
+        </geometry>
+        <material name="chassis"/>
+      </visual>
+      <xacro:box_inertial mass="${mass}" x="${lenght}" y="${width}" z="${height}">
+        <origin xyz="${-axle_offset} 0 0" rpy="0 0 0" />
+      </xacro:box_inertial>
+    </link>
+    <joint name="${name}_joint" type="fixed">
+      <parent link="${robot_name}/base_footprint"/>
+      <child link="${name}_link"/>
+      <origin xyz="0 0 ${height/2.0 + clearence}" rpy="0 0 0"/>
+    </joint>
+  </xacro:macro>
+  <!-- Caster wheel joint and Link definition MACRO -->
+  <xacro:macro name="caster" params="name radius mass offset dx">
+    <link name="${name}_rotation_link">
+      <collision>
+        <origin xyz="${-offset/2.0} 0 0" rpy="0 0 0" />
+        <geometry>
+          <box size="${offset} ${radius} ${radius}"/>
+        </geometry>
+      </collision>
+      <visual>
+        <origin xyz="${-offset/2.0} 0 0" rpy="0 0 0" />
+        <geometry>
+          <box size="${offset} ${radius} ${radius}"/>
+        </geometry>
+        <material name="white"/>
+      </visual>
+      <xacro:box_inertial mass="${mass*0.5}" x="${offset}" y="${radius}" z="${radius}">
+        <origin xyz="${-offset/2.0} 0 0" rpy="0 0 0" />
+      </xacro:box_inertial>
+    </link>
+    <joint name="${name}_rotation_joint" type="continuous">
+      <parent link="${robot_name}/base_footprint"/>
+      <child link="${name}_rotation_link"/>
+      <origin xyz="${dx} 0 ${1.5*caster_radius}" rpy="0 0 0"/>
+      <axis xyz="0 0 1"/>
+      <dynamics damping="0.01" friction="0.1"/>
+    </joint>
+    <link name="${name}_wheel_link">
+      <collision>
+        <origin xyz="0 0 0" rpy="0 0 0"/>
+        <geometry>
+          <sphere radius="${radius}"/>
+        </geometry>
+      </collision>
+      <visual>
+        <origin xyz="0 0 0" rpy="0 0 0"/>
+        <geometry>
+          <sphere radius="${radius}"/>
+        </geometry>
+        <material name="wheel"/>
+      </visual>
+      <xacro:sphere_inertial mass="${mass*0.5}" radius="${radius}">
+        <origin xyz="0 0 0" rpy="0 0 0" />
+      </xacro:sphere_inertial>
+    </link>
+    <joint name="${name}_wheel_joint" type="continuous">
+      <parent link="${name}_rotation_link"/>
+      <child link="${name}_wheel_link"/>
+      <origin xyz="${-offset} 0 ${-caster_radius / 2.0}" rpy="${-PI/2.0} 0 0"/>
+      <axis xyz="0 0 1"/>
+      <dynamics damping="0.01" friction="1.5"/>
+    </joint>
+  </xacro:macro>
 </robot>

File: sr_description/urdf/sr_robot.xacro (robot description, xacro)
@@ -1,9 +1,9 @@
 <?xml version="1.0"?>
-<robot name="sr_robot" xmlns:xacro="http://www.ros.org/wiki/xacro">
-  <!-- Import macros -->
+<robot name="$(arg robot_name)"
+  xmlns:xacro="http://www.ros.org/wiki/xacro">
   <xacro:arg name="robot_name" default="sr_robot"/>
+  <xacro:arg name="update_rate" default="20.0"/>
   <xacro:property name="robot_name" value="$(arg robot_name)"/>
-  <xacro:include filename="$(find sr_description)/urdf/macros.xacro" />
-  <xacro:include filename="$(find sr_description)/urdf/sr_robot.gazebo" />
+  <xacro:property name="update_rate" value="$(arg update_rate)"/>
   <!-- Constants -->
   <xacro:property name="PI" value="3.1415926535897931"/>
@@ -14,5 +14,5 @@
   <!-- Chassis constants -->
   <xacro:property name="chassis_mass" value="12"/>
-  <xacro:property name="chassis_lenght" value="0.95"/>
+  <xacro:property name="chassis_lenght" value="0.75"/>
   <xacro:property name="chassis_width" value="0.5"/>
   <xacro:property name="chassis_height" value="0.3"/>
@@ -26,34 +26,12 @@
   <xacro:property name="caster_radius" value="${clearence/2.0}"/>
   <xacro:property name="caster_offset" value="${caster_radius*1.5}"/>
+  <!-- Import macros -->
+  <xacro:include filename="$(find sr_description)/urdf/macros.xacro" />
   <!-- Robot links -->
   <link name="${robot_name}/base_footprint"/>
-  <xacro:chassis name="${robot_name}/base"
-    mass="${chassis_mass}"
-    lenght="${chassis_lenght}"
-    width="${chassis_width}"
-    height="${chassis_height}"
-    clearence="${clearence}"
-    axle_offset="${axle_offset}"
-  />
-  <xacro:wheel name="${robot_name}/wheel_left"
-    mass="${wheel_mass}"
-    radius="${wheel_radius}"
-    width="${wheel_width}"
-    dx="0"
-    dy="${separation/2.0}"
-  />
-  <xacro:wheel name="${robot_name}/wheel_right"
-    radius="${wheel_radius}"
-    width="${wheel_width}"
-    mass="${wheel_mass}"
-    dx="0"
-    dy="-${separation/2.0}"
-  />
-  <xacro:caster name="${robot_name}/caster"
-    radius="${caster_radius}"
-    mass="${caster_mass}"
-    offset="${caster_offset}"
-    dx="${caster_radius+caster_offset-chassis_lenght/2.0-axle_offset}"
-  />
+  <xacro:chassis name="${robot_name}/base" mass="${chassis_mass}" lenght="${chassis_lenght}" width="${chassis_width}" height="${chassis_height}" clearence="${clearence}" axle_offset="${axle_offset}" />
+  <xacro:wheel name="${robot_name}/wheel_left" mass="${wheel_mass}" radius="${wheel_radius}" width="${wheel_width}" dx="0" dy="${separation/2.0}" />
+  <xacro:wheel name="${robot_name}/wheel_right" radius="${wheel_radius}" width="${wheel_width}" mass="${wheel_mass}" dx="0" dy="-${separation/2.0}" />
+  <xacro:caster name="${robot_name}/caster" radius="${caster_radius}" mass="${caster_mass}" offset="${caster_offset}" dx="${caster_radius+caster_offset-chassis_lenght/2.0-axle_offset}" />
   <!-- IMU -->
   <link name="${robot_name}/imu_link" />
@@ -70,3 +48,10 @@
     <origin xyz="${chassis_lenght/2.0-axle_offset+0.05} 0.0 0.0" rpy="0 0 0" />
   </joint>
+  <link name="${robot_name}/lidar_link"/>
+  <joint name="${robot_name}/lidar_joint" type="fixed">
+    <parent link="${robot_name}/base_link" />
+    <child link="${robot_name}/lidar_link"/>
+    <origin xyz="${chassis_lenght/2.0-axle_offset+0.05} 0.0 0.5" rpy="0 0 0"/>
+  </joint>
+  <xacro:include filename="$(find sr_description)/urdf/sr_robot.gazebo" />
 </robot>
