Commit message: Sync commit

File: sr_description/urdf/sr_robot.xacro (robot description, xacro)
@@ -9,19 +9,19 @@
   <xacro:property name="PI" value="3.1415926535897931"/>
   <!-- Wheels constants -->
-  <xacro:property name="wheel_mass" value="8"/>
-  <xacro:property name="wheel_radius" value="0.25"/>
-  <xacro:property name="wheel_width" value="0.1"/>
+  <xacro:property name="wheel_mass" value="1"/>
+  <xacro:property name="wheel_radius" value="0.125"/>
+  <xacro:property name="wheel_width" value="0.05"/>
   <!-- Chassis constants -->
-  <xacro:property name="chassis_mass" value="12"/>
-  <xacro:property name="chassis_lenght" value="0.75"/>
-  <xacro:property name="chassis_width" value="0.5"/>
-  <xacro:property name="chassis_height" value="0.3"/>
+  <xacro:property name="chassis_mass" value="3"/>
+  <xacro:property name="chassis_lenght" value="0.4"/>
+  <xacro:property name="chassis_width" value="0.25"/>
+  <xacro:property name="chassis_height" value="0.15"/>
   <!-- Robot constants -->
   <xacro:property name="clearence" value="${(wheel_radius-chassis_height/2.0)}"/>
-  <xacro:property name="separation" value="${chassis_width+wheel_width+0.05}"/>
+  <xacro:property name="separation" value="${chassis_width+wheel_width+0.01}"/>
   <xacro:property name="axle_offset" value="${chassis_lenght/2-wheel_radius}"/>
   <!-- <xacro:property name="axle_offset" value="0"/> -->
   <!-- Caster wheel -->
-  <xacro:property name="caster_mass" value="8"/>
+  <xacro:property name="caster_mass" value="0.12"/>
   <xacro:property name="caster_radius" value="${clearence/2.0}"/>
   <xacro:property name="caster_offset" value="${caster_radius*1.5}"/>
